Commit message: Update payload URDF, stair world launch, and patient stairs world

File: ros2_ws/src/go2_with_payload/urdf/go2_with_payload.urdf.xacro (robot description, xacro)
@@ -1,10 +1,8 @@
 <?xml version="1.0"?>
 <robot xmlns:xacro="http://www.ros.org/wiki/xacro" name="go2_with_payload">
-  <!-- rl_sar의 Go2 base xacro include -->
   <xacro:include filename="$(find go2_description)/xacro/robot.xacro"/>
-  <!-- ===== D435i Camera ===== -->
   <link name="d435i_link">
     <inertial>
-      <mass value="0.072"/>
+      <mass value="0.010"/>
       <inertia ixx="0.0001" ixy="0" ixz="0"
                iyy="0.0001" iyz="0" izz="0.0001"/>
@@ -29,8 +27,7 @@
     <origin xyz="0.1423 0 0.2035" rpy="0 0 0"/>
   </joint>
-  <!-- ===== Hesai XT16 LiDAR ===== -->
   <link name="hesai_link">
     <inertial>
-      <mass value="0.830"/>
+      <mass value="0.010"/>
       <inertia ixx="0.001" ixy="0" ixz="0"
                iyy="0.001" iyz="0" izz="0.0005"/>
@@ -55,8 +52,47 @@
     <origin xyz="0.1423 0 0.115" rpy="0 0 0"/>
   </joint>
-  <!-- ===== Oxygen Tank ===== -->
+  <gazebo reference="hesai_link">
+    <sensor type="ray" name="hesai_sensor">
+      <pose>0 0 0 0 0 0</pose>
+      <visualize>false</visualize>
+      <update_rate>10</update_rate>
+      <ray>
+        <scan>
+          <horizontal>
+            <samples>1800</samples>
+            <resolution>1</resolution>
+            <min_angle>-3.14159</min_angle>
+            <max_angle>3.14159</max_angle>
+          </horizontal>
+          <vertical>
+            <samples>16</samples>
+            <resolution>1</resolution>
+            <min_angle>-0.2618</min_angle>
+            <max_angle>0.2618</max_angle>
+          </vertical>
+        </scan>
+        <range>
+          <min>0.3</min>
+          <max>30</max>
+          <resolution>0.01</resolution>
+        </range>
+        <noise>
+          <type>gaussian</type>
+          <mean>0.0</mean>
+          <stddev>0.01</stddev>
+        </noise>
+      </ray>
+      <plugin name="hesai_lidar_controller" filename="libgazebo_ros_ray_sensor.so">
+        <ros>
+          <namespace>/hesai</namespace>
+        </ros>
+        <output_type>sensor_msgs/PointCloud2</output_type>
+        <frame_name>hesai_link</frame_name>
+      </plugin>
+    </sensor>
+  </gazebo>
   <link name="oxygen_tank_link">
     <inertial>
-      <mass value="0.150"/>
+      <mass value="0.010"/>
       <inertia ixx="0.0005" ixy="0" ixz="0"
                iyy="0.0005" iyz="0" izz="0.0005"/>
@@ -81,6 +117,4 @@
     <origin xyz="-0.045 0 0.149" rpy="0 0 0"/>
   </joint>
-  <!-- ===== Sensors (Gazebo plugins) ===== -->
-  <!-- D435i: RGB + Depth -->
   <gazebo reference="d435i_link">
     <sensor type="depth" name="d435i_sensor">
@@ -88,23 +122,9 @@
       <camera>
         <horizontal_fov>1.5708</horizontal_fov>
-        <image>
-          <width>640</width>
-          <height>480</height>
-          <format>R8G8B8</format>
-        </image>
-        <clip>
-          <near>0.1</near>
-          <far>10</far>
-        </clip>
+        <image><width>640</width><height>480</height><format>R8G8B8</format></image>
+        <clip><near>0.1</near><far>10</far></clip>
       </camera>
       <plugin name="d435i_controller" filename="libgazebo_ros_camera.so">
-        <ros>
-          <namespace>/d435i</namespace>
-          <remapping>image_raw:=color/image_raw</remapping>
-          <remapping>image_depth:=depth/image_raw</remapping>
-          <remapping>camera_info:=color/camera_info</remapping>
-          <remapping>camera_info_depth:=depth/camera_info</remapping>
-          <remapping>points:=depth/points</remapping>
-        </ros>
+        <ros><namespace>/d435i</namespace></ros>
         <camera_name>d435i</camera_name>
         <frame_name>d435i_link</frame_name>
@@ -112,36 +132,3 @@
     </sensor>
   </gazebo>
-  <!-- Hesai LiDAR -->
-  <gazebo reference="hesai_link">
-    <sensor type="ray" name="hesai_sensor">
-      <update_rate>10</update_rate>
-      <ray>
-        <scan>
-          <horizontal>
-            <samples>1800</samples>
-            <resolution>1</resolution>
-            <min_angle>-3.14159</min_angle>
-            <max_angle>3.14159</max_angle>
-          </horizontal>
-          <vertical>
-            <samples>16</samples>
-            <resolution>1</resolution>
-            <min_angle>-0.2618</min_angle>
-            <max_angle>0.2618</max_angle>
-          </vertical>
-        </scan>
-        <range>
-          <min>0.3</min>
-          <max>30</max>
-        </range>
-      </ray>
-      <plugin name="hesai_controller" filename="libgazebo_ros_velodyne_laser.so">
-        <ros>
-          <namespace>/hesai</namespace>
-          <remapping>~/out:=points</remapping>
-        </ros>
-        <frame_name>hesai_link</frame_name>
-      </plugin>
-    </sensor>
-  </gazebo>
 </robot>

Commit message: env + waypoint

File: ros2_ws/src/go2_with_payload/urdf/go2_with_payload.urdf.xacro (robot description, xacro)
@@ -4,5 +4,5 @@
   <link name="d435i_link">
     <inertial>
-      <mass value="0.010"/>
+      <mass value="0.001"/>
       <inertia ixx="0.0001" ixy="0" ixz="0"
                iyy="0.0001" iyz="0" izz="0.0001"/>
@@ -29,5 +29,5 @@
   <link name="hesai_link">
     <inertial>
-      <mass value="0.010"/>
+      <mass value="0.001"/>
       <inertia ixx="0.001" ixy="0" ixz="0"
                iyy="0.001" iyz="0" izz="0.0005"/>
@@ -94,5 +94,5 @@
   <link name="oxygen_tank_link">
     <inertial>
-      <mass value="0.010"/>
+      <mass value="0.001"/>
       <inertia ixx="0.0005" ixy="0" ixz="0"
                iyy="0.0005" iyz="0" izz="0.0005"/>
