Commit message: still patient is not on the right waypoint, but no error, still working on the waypoint z

File: ros2_ws/src/patient_simulator/urdf/biped.urdf.xacro (robot description, xacro)
@@ -5,11 +5,11 @@
   <xacro:property name="pelvis_h" value="0.20"/>
   <xacro:property name="pelvis_d" value="0.18"/>
-  <xacro:property name="thigh_length" value="0.42"/>
+  <xacro:property name="thigh_length" value="0.38"/>
   <xacro:property name="thigh_radius" value="0.08"/>
-  <xacro:property name="shank_length" value="0.42"/>
+  <xacro:property name="shank_length" value="0.38"/>
   <xacro:property name="shank_radius" value="0.06"/>
-  <xacro:property name="foot_length" value="0.25"/>
-  <xacro:property name="foot_width" value="0.12"/>
-  <xacro:property name="foot_height" value="0.05"/>
+  <xacro:property name="foot_length" value="0.20"/>
+  <xacro:property name="foot_width" value="0.09"/>
+  <xacro:property name="foot_height" value="0.04"/>
   <xacro:property name="hip_offset_y" value="0.10"/>
   <xacro:macro name="box_inertia" params="m x y z">
@@ -63,12 +63,4 @@
       <material name="dark_gray"><color rgba="0.3 0.3 0.3 1"/></material>
     </visual>
-    <collision>
-      <geometry><box size="${pelvis_d} ${pelvis_w} ${pelvis_h}"/></geometry>
-    </collision>
-    <visual name="head">
-      <origin xyz="0 0 ${pelvis_h/2 + 0.15}" rpy="0 0 0"/>
-      <geometry><sphere radius="0.10"/></geometry>
-      <material name="skin"><color rgba="0.9 0.7 0.6 1"/></material>
-    </visual>
   </link>
   <xacro:macro name="leg" params="side reflect">
@@ -91,8 +83,4 @@
         <material name="blue"><color rgba="0.2 0.2 0.7 1"/></material>
       </visual>
-      <collision>
-        <origin xyz="0 0 ${-thigh_length/2}"/>
-        <geometry><cylinder radius="${thigh_radius}" length="${thigh_length}"/></geometry>
-      </collision>
     </link>
     <joint name="${side}_knee_joint" type="revolute">
@@ -114,8 +102,4 @@
         <material name="blue"/>
       </visual>
-      <collision>
-        <origin xyz="0 0 ${-shank_length/2}"/>
-        <geometry><cylinder radius="${shank_radius}" length="${shank_length}"/></geometry>
-      </collision>
     </link>
     <joint name="${side}_ankle_joint" type="revolute">
@@ -137,8 +121,4 @@
         <material name="black"><color rgba="0.1 0.1 0.1 1"/></material>
       </visual>
-      <collision>
-        <origin xyz="${foot_length/4} 0 ${-foot_height/2}"/>
-        <geometry><box size="${foot_length} ${foot_width} ${foot_height}"/></geometry>
-      </collision>
     </link>
   </xacro:macro>

Commit message: /odom work, yolo detector target_vaild true, patient p3d plugin

File: ros2_ws/src/patient_simulator/urdf/biped.urdf.xacro (robot description, xacro)
@@ -63,4 +63,24 @@
       <material name="dark_gray"><color rgba="0.3 0.3 0.3 1"/></material>
     </visual>
+    <visual name="torso">
+      <origin xyz="0 0 ${pelvis_h/2 + 0.30}" rpy="0 0 0"/>
+      <geometry><box size="0.20 0.40 0.60"/></geometry>
+      <material name="torso_clr"><color rgba="0.5 0.3 0.2 1"/></material>
+    </visual>
+    <visual name="head">
+      <origin xyz="0 0 ${pelvis_h/2 + 0.75}" rpy="0 0 0"/>
+      <geometry><sphere radius="0.12"/></geometry>
+      <material name="skin"><color rgba="0.9 0.7 0.6 1"/></material>
+    </visual>
+    <visual name="left_arm">
+      <origin xyz="0 0.25 ${pelvis_h/2 + 0.30}" rpy="0 0 0"/>
+      <geometry><cylinder radius="0.05" length="0.55"/></geometry>
+      <material name="arm_clr"><color rgba="0.5 0.3 0.2 1"/></material>
+    </visual>
+    <visual name="right_arm">
+      <origin xyz="0 -0.25 ${pelvis_h/2 + 0.30}" rpy="0 0 0"/>
+      <geometry><cylinder radius="0.05" length="0.55"/></geometry>
+      <material name="arm_clr"/>
+    </visual>
   </link>
   <xacro:macro name="leg" params="side reflect">
@@ -186,3 +206,15 @@
     </plugin>
   </gazebo>
+<gazebo>
+  <plugin name="patient_p3d" filename="libgazebo_ros_p3d.so">
+    <ros>
+      <namespace>/patient</namespace>
+      <remapping>odom:=odom</remapping>
+    </ros>
+    <update_rate>50</update_rate>
+    <body_name>pelvis_link</body_name>
+    <frame_name>world</frame_name>
+    <gaussian_noise>0.0</gaussian_noise>
+  </plugin>
+</gazebo>
 </robot>
