Commit message: change color, good but not follow oodm not working

File: ros2_ws/src/patient_simulator/urdf/biped.urdf.xacro (robot description, xacro)
@@ -2,4 +2,8 @@
 <robot xmlns:xacro="http://www.ros.org/wiki/xacro" name="biped_patient">
   <material name="dark_gray"><color rgba="0.3 0.3 0.3 1"/></material>
+  <material name="skin"><color rgba="0.9 0.75 0.65 1"/></material>
+  <material name="shirt"><color rgba="0.2 0.4 0.7 1"/></material>
+  <material name="pants"><color rgba="0.15 0.15 0.35 1"/></material>
+  <material name="shoes"><color rgba="0.4 0.3 0.2 1"/></material>
   <link name="world"/>
   <link name="base_x_link">
@@ -45,5 +49,5 @@
     <parent link="base_z_link"/>
     <child link="pelvis_link"/>
-    <origin xyz="0 0 1.0242" rpy="0 0 0"/>
+    <origin xyz="0 0 1.06" rpy="0 0 0"/>
     <axis xyz="0 1 0"/>
     <limit lower="-1.57" upper="1.57" effort="1000" velocity="10"/>
@@ -178,5 +182,5 @@
     <parent link="pelvis_link"/>
     <child link="torso_link"/>
-    <origin xyz="0 0 0" rpy="0 0 0"/>
+    <origin xyz="0 0 -0.25" rpy="0 0 0"/>
   </joint>
   <link name="L_shoulder_pitch_link">
@@ -341,3 +345,74 @@
     </plugin>
   </gazebo>
+  <!-- Gazebo material overrides -->
+  <gazebo reference="pelvis_link">
+    <material>Gazebo/Black</material>
+    <gravity>false</gravity>
+  </gazebo>
+  <gazebo reference="torso_link">
+    <material>Gazebo/Black</material>
+    <gravity>false</gravity>
+  </gazebo>
+  <gazebo reference="L_thigh_link">
+    <material>Gazebo/Black</material>
+    <gravity>false</gravity>
+  </gazebo>
+  <gazebo reference="L_shank_link">
+    <material>Gazebo/Black</material>
+    <gravity>false</gravity>
+  </gazebo>
+  <gazebo reference="L_foot_link">
+    <material>Gazebo/Black</material>
+    <gravity>false</gravity>
+  </gazebo>
+  <gazebo reference="R_thigh_link">
+    <material>Gazebo/Black</material>
+    <gravity>false</gravity>
+  </gazebo>
+  <gazebo reference="R_shank_link">
+    <material>Gazebo/Black</material>
+    <gravity>false</gravity>
+  </gazebo>
+  <gazebo reference="R_foot_link">
+    <material>Gazebo/Black</material>
+    <gravity>false</gravity>
+  </gazebo>
+  <gazebo reference="L_shoulder_pitch_link">
+    <material>Gazebo/Black</material>
+    <gravity>false</gravity>
+  </gazebo>
+  <gazebo reference="L_shoulder_roll_link">
+    <material>Gazebo/Black</material>
+    <gravity>false</gravity>
+  </gazebo>
+  <gazebo reference="L_shoulder_yaw_link">
+    <material>Gazebo/Black</material>
+    <gravity>false</gravity>
+  </gazebo>
+  <gazebo reference="L_elbow_link">
+    <material>Gazebo/Black</material>
+    <gravity>false</gravity>
+  </gazebo>
+  <gazebo reference="R_shoulder_pitch_link">
+    <material>Gazebo/Black</material>
+    <gravity>false</gravity>
+  </gazebo>
+  <gazebo reference="R_shoulder_roll_link">
+    <material>Gazebo/Black</material>
+    <gravity>false</gravity>
+  </gazebo>
+  <gazebo reference="R_shoulder_yaw_link">
+    <material>Gazebo/Black</material>
+    <gravity>false</gravity>
+  </gazebo>
+  <gazebo reference="R_elbow_link">
+    <material>Gazebo/Black</material>
+    <gravity>false</gravity>
+  </gazebo>
+  <gazebo reference="base_x_link">
+    <gravity>false</gravity>
+  </gazebo>
+  <gazebo reference="base_z_link">
+    <gravity>false</gravity>
+  </gazebo>
 </robot>
